File: vizszintkapcs_v1_4.brd (EAGLE design)
At the start: 238.3 x 119.9 mm, 168 parts, among them IC2 7815TV, J10 PWR, J3 PWR, Q2 32.768kHz, Q4 CSTCR4M00G15L99, U1 MCP3004-I/ST, U6 MSP430F5529IPNR

Commit message: without MCU
Parts:
- removed C15, C16: 220n, rcl:0402
- removed C17: 1n, rcl:0402
- removed C18: 470n, rcl:0402
- removed C19, C20, C21, C29: 100n, rcl:0402
- removed C23, C24: 10p, rcl:0402
- removed C25, C26: 12p, rcl:0402
- removed C27: 4u7, rcl:A/3216-18R
- removed C30: 10u, rcl:A/3216-18R
- removed H1, H2: MOUNT-PAD-SQUARE4.1, holes:4,1-PAD-SQUARE
- removed J10, J3: PWR, pinhead:1X03
- removed JP1: +5V, jumper:JP1M
- removed JP10, JP12, JP5, JP6, JP7, JP9: (no value), SparkFun:1X02
- removed JP11: USB-A-H, SparkFun-Connectors:USB-A-H
- removed JP2: +3V3, jumper:JP1M
- removed JP3: GND, jumper:JP1M
- removed JP4: (no value), pinhead-1:1X02M
- removed JP4.1: SBW_TST, jumper:JP1M
- removed JP4.2: SBW_RST, jumper:JP1M
- removed JP4.3: SBW_NC, jumper:JP1M
- removed JP6.1: TXD, jumper:JP1M
- removed JP6.2: RXD, jumper:JP1M
- removed JP6.3: CTS, jumper:JP1M
- removed JP6.4: RTS, jumper:JP1M
- removed JP8: LED1_PWR, jumper:JP1
- removed LD1117: V_REG_LD1117VXX, SparkFun-PowerIC:78XXL
- removed LED1, LED2: (no value), led:CHIPLED_0603
- removed LSP1, LSP10, LSP2, LSP3, LSP4, LSP5, LSP6, LSP7, LSP8, LSP9, WATERIN: SE14, solpad:SE14
- removed NRF24_MODULE: M04X2, SparkFun-Connectors:2X4
- removed Q2: 32.768kHz, microcrystal:MS3V-T1R
- removed Q4: CSTCR4M00G15L99, murata:MURATA-FILTER_CSTCR
- removed R14: 100R, rcl:0402
- removed R15: 1k4, rcl:0402
- removed R16: 1M, rcl:0402
- removed R27: 47k, rcl:0402
- removed R28: 0R, rcl:0402
- removed R29, R30: 470R, rcl:0402
- removed R31, R32: 27R, rcl:0402
- removed S1, S2: (no value), electricalmeter:PBTH
- removed S3: RST, electricalmeter:PBTH
- removed S4: (no value), adafruit:EG1218
- removed S5: BSL, electricalmeter:PBTH
- removed U6: MSP430F5529IPNR, TI_MSP430_v16_intern:PN80
- removed USB-SERIAL2:C1, USB-SERIAL2:C4: 100nF, SparkFun-Passives:1206
- removed USB-SERIAL2:C3: 4.7uF, SparkFun-Passives:EIA3216
- removed USB-SERIAL2:JP2: (no value), SparkFun-Connectors:1X03
- removed USB-SERIAL2:LED1, USB-SERIAL2:LED2: (no value), SparkFun-LED:FKIT-LED-1206
- removed USB-SERIAL2:R1, USB-SERIAL2:R2: 400, SparkFun-Resistors:1206
- removed USB-SERIAL2:U1: FT232RL-BASICSSOP, SparkFun-DigitalIC:SSOP28DB
- added IC1: UA78M08DCY, linear:SOT223
- added U$2: STMICRO_L7808, forCNC:TO220S
- added U$3: TERMINAL_BLOCK_4:METZ_AST1350404, forCNC:TERMINAL_BLOCK_4:METZ_AST1350404
- added U$6: TERMINAL_BLOCK_6:METZ_AST1350604, forCNC:TERMINAL_BLOCK_6:METZ_AST1350604
- added U$8: TERMINAL_BLOCK_10:METZ_AST0451004, forCNC:TERMINAL_BLOCK_10:METZ_AST0451004
- 7805: value (none) -> FAIRCHILD_LM7805CT; device SparkFun-PowerIC:TO220-IGO -> forCNC:TO220S
- C5: value 100n -> 470uF; device rcl:0402 -> capacitor-wima:C2.5-3
- C6: value 10uF -> 10nF
- REL_MOT:T1: value BDX53 -> BDX53_STANDING; device transistor:TO220 -> forCNC:TO220S
- moved C11 220.9 mm to (137.2, 25.7)
- moved C8 220.9 mm to (110.7, 18.5)
- moved GPIO_CON1 220.9 mm to (139.7, 12.7)
- moved U$1 220.9 mm to (125.0, 20.8)
- moved U1 220.9 mm to (136.1, 21.3)
- moved WL6:B3 212.4 mm to (174.0, 16.5), turned to 0 degrees
- moved WL5:B3 208.7 mm to (182.9, 16.5), turned to 0 degrees
- moved WL4:B3 205.7 mm to (191.8, 16.5), turned to 0 degrees
- moved WL6:R7 205.6 mm to (174.0, 21.6), turned to 0 degrees
- moved WL3:B3 203.5 mm to (200.7, 16.5), turned to 0 degrees
- moved WL6:C4 202.2 mm to (174.0, 24.1), turned to 180 degrees
- moved WL2:B3 202.0 mm to (209.6, 16.5), turned to 0 degrees
- moved WL5:R7 201.8 mm to (182.9, 21.6), turned to 0 degrees
- moved WL1:B3 201.2 mm to (218.4, 16.5), turned to 0 degrees
- moved WL4:R7 198.7 mm to (191.8, 21.6), turned to 0 degrees
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Connections:
- removed net !CTS: USB-SERIAL2:U1.11
- removed net !DTR: USB-SERIAL2:U1.2
- removed net !RTS: USB-SERIAL2:U1.3
- removed net +3V3: C19.2, C20.1, C30.+, C5.1, J10.3, JP2.2, R27.2, R28.2, S5.1, U6.18, U6.50
- removed net +5V: C21.1, C27.+, J3.3, JP1.2, U6.65
- removed net 7805_DC5V: 7805.OUT, C3.1, C9.1, S4.S
- removed net AVCC: C29.1, R28.1, U6.11
- removed net CE_NRF: JP12.2, NRF24_MODULE.3
- removed net CSN_NRF: JP7.1, NRF24_MODULE.4
- removed net D+: JP11.D+, USB-SERIAL2:U1.15
- removed net D-: JP11.D-, USB-SERIAL2:U1.16
- removed net EZFET_SBW_NC: JP4.3.1
- removed net EZFET_SBW_RST: JP4.2.1
- removed net EZFET_SBW_TST: JP4.1.1
- removed net EZFET_UARTCTS: JP6.4.1
- removed net EZFET_UARTRTS: JP6.3.1
- removed net EZFET_UARTRXD: JP6.1.1, USB-SERIAL2:U1.5
- removed net EZFET_UARTTXD: JP6.2.1, USB-SERIAL2:U1.1
- removed net HUB_DM1: JP4.1, R31.1
- removed net HUB_DP1: JP4.2, R32.1
- removed net IRQ_NRF: JP6.1, NRF24_MODULE.8
- removed net MISO_NRF: JP10.2, NRF24_MODULE.7
- removed net MOSI_NRF: JP5.1, NRF24_MODULE.6
- removed net N$32: LED1.A, R29.2
- removed net N$35: LED2.A, R30.2
- removed net N$4: R14.1, S5.2
- removed net N$7: JP8.2, R29.1
- removed net P1.0: JP8.1, U6.21
- removed net P1.1: S2.1, U6.22
- removed net P1.2: JP6.2, U6.23
- removed net P1.7: JP6.3.2, U6.28
- removed net P2.0: U6.29
- removed net P2.1: S1.1, U6.30
- removed net P2.2: U6.31
- removed net P2.3: JP12.1, U6.32
- removed net P2.6: U6.35
- removed net P3.0: JP5.2, U6.37
- removed net P3.1: JP10.1, U6.38
- removed net P3.2: JP9.1, U6.39
- removed net P3.3: U6.40
- removed net P3.4: U6.41
- removed net P3.5: U6.42
- removed net P3.6: U6.43
- removed net P3.7: U6.44
- removed net P4.0: U6.45
- removed net P4.1: U6.46
- removed net P4.2: U6.47
- removed net P4.4/UCA1TXD: JP6.1.2, U6.51
- removed net P4.5/UCA1RXD: JP6.2.2, U6.52
- removed net P4.7: R30.1, U6.54
- removed net P5.2/XT2IN: Q4.3, U6.69
- removed net P5.3/XT2OUT: Q4.1, U6.70
- removed net P5.4/XIN: C26.2, Q2.P2, U6.12
- removed net P5.5/XOUT: C25.2, Q2.P1, U6.13
- removed net P6.2: U6.79
- removed net P6.3: U6.80
- removed net P6.4: U6.1
- removed net P6.5: U6.2
- removed net P6.6: U6.3
- removed net P6.7: JP6.4.2, U6.4
- removed net P7.0: U6.5
- removed net P7.4: U6.57
- removed net P8.1: U6.16
- removed net P8.2: U6.17
- removed net RST/SBWTDIO: C17.1, JP4.2.2, R27.1, S3.2, U6.76
- removed net SCK_NRF: JP9.2, NRF24_MODULE.5
- removed net TARGET_DM: C24.1, R31.2, U6.64
- removed net TARGET_DP: C23.1, R15.2, R32.2, U6.62
- removed net TARGET_PUR: R14.2, R15.1, R16.2, U6.63
- removed net TARGET_VUSB: C16.1, U6.66
- removed net TEST/SBWTCK: JP4.1.2, U6.71
- removed net USB-SERIAL2:3V3FTDI: USB-SERIAL2:C4.1, USB-SERIAL2:JP2.1, USB-SERIAL2:U1.17
- removed net USB-SERIAL2:N$1: USB-SERIAL2:LED1.C, USB-SERIAL2:U1.22
- removed net USB-SERIAL2:N$2: USB-SERIAL2:LED2.C, USB-SERIAL2:U1.23
- removed net USB-SERIAL2:N$3: USB-SERIAL2:LED2.A, USB-SERIAL2:R1.1
- removed net USB-SERIAL2:N$4: USB-SERIAL2:LED1.A, USB-SERIAL2:R2.1
- removed net USB-SERIAL2:VCCIO: USB-SERIAL2:JP2.2, USB-SERIAL2:U1.4
- removed net USB_5V: JP11.VBUS, S4.O
- removed net V18: C15.1, U6.67
- removed net VCC: USB-SERIAL2:C1.1, USB-SERIAL2:C3.A, USB-SERIAL2:JP2.3, USB-SERIAL2:R1.2, USB-SERIAL2:R2.2, USB-SERIAL2:U1.20
- removed net VCORE: C18.2, U6.20
- new net COMMON_EARTH: U$8.P$10, U$8.P$2, U$8.P$5, U$8.P$8
- new net DC8V: C5.1, C6.1, U$2.3, U$3.P$4
- net 1_WATER_IN: now also U$6.P$1; no longer LSP5.MP
- net 230V0: now also U$8.P$3; no longer H2.B4,1
- net 230VPHASE: now also U$8.P$1; no longer H1.B4,1
- net 2_WATER_IN: now also U$6.P$2; no longer LSP6.MP
- net 3_WATER_IN: now also U$6.P$3; no longer LSP7.MP
- net 4_WATER_IN: now also U$6.P$4; no longer LSP8.MP
- net 5_WATER_IN: now also U$6.P$5; no longer LSP9.MP
- net 6_WATER_IN: now also U$6.P$6; no longer LSP10.MP
- net AC12V: now also U$3.P$2; no longer WATERIN.MP
- net DC3.3V: now also IC1.3; no longer C6.2, JP2.1, LD1117.GND, NRF24_MODULE.2
- net DC5V: now also 7805.3, C3.1, C9.1; no longer JP1.1, LD1117.OUT, S4.P
- net GND: now also 7805.2, C6.2, IC1.2, IC1.4, U$2.2, U$3.P$3; no longer 7805.GND, C15.2, C16.2, C17.2, C18.1, C19.1, C20.2, C21.2, C23.2, C24.2, C25.1, C26.1, C27.-, C29.2, C30.-, C6.1, J10.1, J10.2, J3.1, J3.2, JP11.GND, JP3.1, JP3.2, LD1117.IN, LED1.C, LED2.C, NRF24_MODULE.1, Q2.P3, Q4.2, R16.1, S1.2, S2.2, S3.1, U6.14, U6.19, U6.49, U6.61, U6.68, USB-SERIAL2:C1.2, USB-SERIAL2:C3.C, USB-SERIAL2:C4.2, USB-SERIAL2:U1.18, USB-SERIAL2:U1.21, USB-SERIAL2:U1.25, USB-SERIAL2:U1.26, USB-SERIAL2:U1.7
- net MOTOR_DIRECT_1: now also U1.1; no longer U1.3
- net MOTOR_DIRECT_2: now also U1.3; no longer U1.4
- net MOTOR_IN: now also SSR_MOT:K1.1, SSR_MOT:R2.P$1, U$8.P$4; no longer LSP1.MP, SSR_MOT:C1.1, SSR_MOT:U$1.3, SSR_MOT:U$1.4
- net MOTOR_IN_2: now also REL_MOT:K1.S1, REL_MOT:R2.P$1, U$8.P$7; no longer LSP3.MP, REL_MOT:C1.1, REL_MOT:U$1.3, REL_MOT:U$1.4
- net MOTOR_OUT_1: now also SSR_MOT:C1.1, SSR_MOT:U$1.3, SSR_MOT:U$1.4, U$8.P$6; no longer LSP2.MP, SSR_MOT:K1.1, SSR_MOT:R2.P$1
- net MOTOR_OUT_2: now also REL_MOT:C1.1, REL_MOT:U$1.3, REL_MOT:U$1.4, U$8.P$9; no longer LSP4.MP, REL_MOT:K1.S1, REL_MOT:R2.P$1
- net P1.3: no longer U6.24
- net P1.4: no longer U6.25
- net P1.5: no longer U6.26
- net P1.6: no longer U6.27
- net P2.4: no longer JP7.2, U6.33
- net P2.5: no longer U6.34
- net P2.7: no longer U6.36
- net P4.3: no longer U6.48
- net P6.0: now also U1.4; no longer U1.2, U6.77
- net P6.1: now also U1.2; no longer U1.1, U6.78
- net REC12V: now also 7805.1, IC1.1; no longer 7805.IN
- net REC24V: now also U$2.1
Routing:
- net P1.6: track 277.8 -> 86.9 mm, vias 3 -> 1
- net 230VPHASE: track 66.0 -> 253.7 mm, vias 0 -> 1
- net P6.1: track 299.9 -> 115.9 mm, vias 4 -> 0
- net P6.0: track 283.7 -> 138.9 mm, vias 6 -> 0
- net DC8V: track 0.00 -> 126.4 mm, vias 0 -> 3
- net +3V3: track 120.4 -> 0.00 mm, vias 6 -> 0
- net DC3.3V: track 176.0 -> 66.2 mm, vias 3 -> 0
- net +5V: track 107.1 -> 0.00 mm, vias 6 -> 0
- net MOTOR_DIRECT_1: track 211.9 -> 126.1 mm, vias 4 -> 2
- net TRANS_OUT: track 254.5 -> 170.8 mm
- net VCC: track 72.4 -> 0.00 mm
- net P2.4: track 126.3 -> 56.6 mm, vias 4 -> 0
- net P1.3: track 146.1 -> 76.7 mm, vias 4 -> 0
- net P4.3: track 149.3 -> 82.2 mm, vias 2 -> 0
- net RST/SBWTDIO: track 60.2 -> 0.00 mm, vias 2 -> 0
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Other:
- board size 238.3 x 119.9 mm -> 235.7 x 107.2 mm
- board text added: "230V0"
- board text added: "230VACT"
- board text added: "AC12v"
- board text added: "DC8V"
- board text added: "MOTOR1 IN"
- board text added: "MOTOR1 OUT"
- board text added: "MOTOR2 IN"
- board text added: "MOTOR2 OUT"
- board text added: "Olinuxino hole"
- board text added: "PE"
- board text added: "WATER LEVEL SENSORS"
