File: vizszintkapcs_v1_4.sch (EAGLE design)
At the start: 27 parts, among them IC1 UA78M33DCY, IC2 7815TV, U1 MCP3004-I/ST

Commit message: 3.3v spi levels
Connections:
- net DC3.3V: now also C11.1, C8.1, U$1.VDD, U1.VDD, U1.VREF
- net DC5V: no longer C11.1, C8.1, U$1.VDD, U1.VDD, U1.VREF
Changed lines of the file:
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@@
-</segment>
-<segment>
-<pinref part="U1" gate="A" pin="VDD"/>
-<wire x1="383.54" y1="190.5" x2="365.76" y2="190.5" width="0.1524" layer="91"/>
-<label x="370.84" y="190.5" size="1.778" layer="95"/>
-<wire x1="365.76" y1="190.5" x2="365.76" y2="193.04" width="0.1524" layer="91"/>
-<pinref part="C8" gate="G$1" pin="1"/>
-<wire x1="365.76" y1="193.04" x2="360.68" y2="193.04" width="0.1524" layer="91"/>
-</segment>
-<segment>
-<pinref part="U1" gate="A" pin="VREF"/>
-<wire x1="383.54" y1="195.58" x2="370.84" y2="195.58" width="0.1524" layer="91"/>
-<label x="370.84" y="195.58" size="1.778" layer="95"/>
-</segment>
-<segment>
-<pinref part="C11" gate="G$1" pin="1"/>
-<pinref part="U$1" gate="A" pin="VDD"/>
-<wire x1="360.68" y1="248.92" x2="360.68" y2="256.54" width="0.1524" layer="91"/>
-<wire x1="360.68" y1="256.54" x2="383.54" y2="256.54" width="0.1524" layer="91"/>
-<label x="363.22" y="256.54" size="1.778" layer="95"/>
 </segment>
 <segment>
@@
 <portref moduleinst="WL5" port="VCC"/>
 </segment>
-</net>
+<segment>
+<pinref part="U1" gate="A" pin="VREF"/>
+<wire x1="383.54" y1="195.58" x2="370.84" y2="195.58" width="0.1524" layer="91"/>
+<label x="370.84" y="195.58" size="1.778" layer="95"/>
+</segment>
+<segment>
+<pinref part="C8" gate="G$1" pin="1"/>
+<wire x1="360.68" y1="193.04" x2="368.3" y2="193.04" width="0.1524" layer="91"/>
+<wire x1="368.3" y1="193.04" x2="368.3" y2="190.5" width="0.1524" layer="91"/>
+<pinref part="U1" gate="A" pin="VDD"/>
+<wire x1="368.3" y1="190.5" x2="383.54" y2="190.5" width="0.1524" layer="91"/>
+<label x="370.84" y="190.5" size="1.778" layer="95"/>
+</segment>
+<segment>
+<pinref part="C11" gate="G$1" pin="1"/>
+<wire x1="360.68" y1="248.92" x2="360.68" y2="256.54" width="0.1524" layer="91"/>
+<pinref part="U$1" gate="A" pin="VDD"/>
+<wire x1="360.68" y1="256.54" x2="383.54" y2="256.54" width="0.1524" layer="91"/>
+<label x="360.68" y="256.54" size="1.778" layer="95"/>
+</segment>
+</net>
